Commit message: 0319

File: assets/all_robot/urdfmodel.urdf (robot description, URDF)
Before this commit: robot all_robot, 19 links, 18 joints
Links:
- link left_ee_link: geometry collision cylinder length=0.184 radius=0.025; visual cylinder length=0.184 radius=0.025
- link right_ee_link: geometry collision cylinder length=0.184 radius=0.025; visual cylinder length=0.184 radius=0.025
Joints:
- joint waist_joint: origin xyz=-0.048059 0 0.86826 rpy=-1.5708 0.4014 0 -> xyz=-0.048059 0 0.86826 rpy=-1.5708 0.4835 0

File: assets/right_rm65f/right_rm65.urdf (robot description, URDF)
Before this commit: robot RM65F-R, 10 links, 9 joints
Links:
- link right_ee_link: geometry collision cylinder length=0.184 radius=0.025; visual cylinder length=0.184 radius=0.025

Commit message: 0327

File: assets/all_robot/urdfmodel.urdf (robot description, URDF)
Before this commit: robot all_robot, 19 links, 18 joints
Joints:
- joint waist_joint: origin xyz=-0.048059 0 0.86826 rpy=-1.5708 0.4835 0 -> xyz=-0.048059 0 0.86826 rpy=-1.5708 0.0 0
